Commit message: Clean-up

File: ngeeann_av_description/urdf/camera.xacro (robot description, xacro)
@@ -1,5 +1,4 @@
 <?xml version="1.0" ?>
 <robot name="ngeeann_av" xmlns:xacro="http://www.ros.org/wiki/xacro">
-  <!-- Camera -->
   <joint name="camera_joint" type="fixed">
     <axis xyz="0 0 0" />
@@ -30,3 +29,47 @@
     </inertial>
   </link>
+  <gazebo reference="camera_link">
+		<mu1>0.2</mu1>
+		<mu2>0.2</mu2>
+		<material>Gazebo/Red</material>
+	</gazebo>
+	<gazebo reference="camera_link">
+		<sensor type="camera" name="camera1">
+		  <update_rate>30.0</update_rate>
+		  <camera name="head">
+		    <horizontal_fov>1.3962634</horizontal_fov>
+		    <image>
+		      <width>800</width>
+		      <height>800</height>
+		      <format>R8G8B8</format>
+		    </image>
+		    <clip>
+		      <near>0.02</near>
+		      <far>300</far>
+		    </clip>
+		    <noise>
+		      <type>gaussian</type>
+		      <!-- Noise is sampled independently per pixel on each frame.
+		           That pixel's noise value is added to each of its color
+		           channels, which at that point lie in the range [0,1]. -->
+		      <mean>0.0</mean>
+		      <stddev>0.007</stddev>
+		    </noise>
+		  </camera>
+		  <plugin name="camera_controller" filename="libgazebo_ros_camera.so">
+		    <alwaysOn>true</alwaysOn>
+		    <updateRate>0.0</updateRate>
+		    <cameraName>robot/camera1</cameraName>
+		    <imageTopicName>image_raw</imageTopicName>
+		    <cameraInfoTopicName>camera_info</cameraInfoTopicName>
+		    <frameName>camera_link</frameName>
+		    <hackBaseline>0.07</hackBaseline>
+		    <distortionK1>0.0</distortionK1>
+		    <distortionK2>0.0</distortionK2>
+		    <distortionK3>0.0</distortionK3>
+		    <distortionT1>0.0</distortionT1>
+		    <distortionT2>0.0</distortionT2>
+		  </plugin>
+		</sensor>
+	</gazebo>
 </robot>

File: ngeeann_av_description/urdf/hokuyo.xacro (robot description, xacro)
@@ -26,3 +26,38 @@
 		</inertial>
 	</link>
+	<gazebo reference="hokuyo_link">
+		<sensor type="ray" name="head_hokuyo_sensor">
+		  <pose>0 0 0 0 0 0</pose>
+		  <visualize>true</visualize>
+		  <update_rate>40</update_rate>
+		  <ray>
+		    <scan>
+		      <horizontal>
+		        <samples>720</samples>
+		        <resolution>1</resolution>
+		        <min_angle>-1.570796</min_angle>
+		        <max_angle>1.570796</max_angle>
+		      </horizontal>
+		    </scan>
+		    <range>
+		      <min>0.10</min>
+		      <max>30.0</max>
+		      <resolution>0.01</resolution>
+		    </range>
+		    <noise>
+		      <type>gaussian</type>
+		      <!-- Noise parameters based on published spec for Hokuyo laser
+		             achieving "+-30mm" accuracy at range < 10m.  A mean of 0.0m and
+		             stddev of 0.01m will put 99.7% of samples within 0.03m of the true
+		             reading. -->
+		      <mean>0.0</mean>
+		      <stddev>0.01</stddev>
+		    </noise>
+		  </ray>
+		  <plugin name="gazebo_ros_head_hokuyo_controller" filename="libgazebo_ros_laser.so">
+		    <topicName>/robot/laser/scan</topicName>
+		    <frameName>hokuyo_link</frameName>
+		  </plugin>
+		</sensor>
+	</gazebo>
 </robot>

Commit message: Add files via upload

File: ngeeann_av_description/urdf/camera.xacro (robot description, xacro)
@@ -1,4 +1,5 @@
 <?xml version="1.0" ?>
 <robot name="ngeeann_av" xmlns:xacro="http://www.ros.org/wiki/xacro">
+	<xacro:property name="camera_link" value="0.05" />
   <joint name="camera_joint" type="fixed">
     <axis xyz="0 0 0" />

File: ngeeann_av_description/urdf/ngeeann_av.xacro (robot description, xacro)
@@ -6,5 +6,4 @@
 <xacro:include filename="$(find ngeeann_av_description)/urdf/hokuyo.xacro" />
 <xacro:include filename="$(find ngeeann_av_description)/urdf/camera.xacro" />
-<xacro:property name="camera_link" value="0.05" />
 <link name="base_link">
   <inertial>
@@ -171,5 +170,5 @@
   <axis xyz="-1.0 0.0 0.0"/>
 </joint>
-<joint name="r_steer" type="revolute">
+<joint name="fr_steer" type="revolute">
   <origin rpy="0 0 0" xyz="0.825001 1.517363 -0.144363"/>
   <parent link="base_link"/>
@@ -178,5 +177,5 @@
   <limit effort="1000.0" lower="-0.95" upper="0.95" velocity="5"/>
 </joint>
-<joint name="l_steer" type="revolute">
+<joint name="fl_steer" type="revolute">
   <origin rpy="0 0 0" xyz="-0.824999 1.517363 -0.144363"/>
   <parent link="base_link"/>
@@ -185,3 +184,17 @@
   <limit effort="1000.0" lower="-0.95" upper="0.95" velocity="5"/>
 </joint>
+<joint name="fr_steer" type="revolute">
+  <origin rpy="0 0 0" xyz="0.825001 1.517363 -0.144363"/>
+  <parent link="base_link"/>
+  <child link="r_steer_1"/>
+  <axis xyz="-0.0 -0.0 1.0"/>
+  <limit effort="1000.0" lower="-0.95" upper="0.95" velocity="5"/>
+</joint>
+<joint name="fl_steer" type="revolute">
+  <origin rpy="0 0 0" xyz="-0.824999 1.517363 -0.144363"/>
+  <parent link="base_link"/>
+  <child link="l_steer_1"/>
+  <axis xyz="-0.0 -0.0 1.0"/>
+  <limit effort="1000.0" lower="-0.95" upper="0.95" velocity="5"/>
+</joint>
 </robot>

Commit message: revised base_link

File: ngeeann_av_description/urdf/camera.xacro (robot description, xacro)
@@ -5,5 +5,5 @@
     <axis xyz="0 0 0" />
     <origin xyz="0 2.45 0.07" rpy="0 0 1.5708"/>
-    <parent link="base_link"/>
+    <parent link="chassis_link"/>
     <child link="camera_link"/>
   </joint>

File: ngeeann_av_description/urdf/hokuyo.xacro (robot description, xacro)
@@ -4,5 +4,5 @@
 		<axis xyz="0 1 0" />
 		<origin xyz="0 2.34 0.24" rpy="0 0 1.5708"/>
-		<parent link="base_link"/>
+		<parent link="chassis_link"/>
 		<child link="hokuyo_link"/>
 	</joint>

File: ngeeann_av_description/urdf/ngeeann_av.xacro (robot description, xacro)
@@ -6,5 +6,11 @@
 <xacro:include filename="$(find ngeeann_av_description)/urdf/hokuyo.xacro" />
 <xacro:include filename="$(find ngeeann_av_description)/urdf/camera.xacro" />
-<link name="base_link">
+<link name="base_link"/>
+<joint name="base_link_joint" type="fixed">
+  <origin xyz="0 0 0.46936" rpy="0 0 0" />
+  <parent link="base_link"/>
+  <child link="chassis_link"/>
+</joint>
+<link name="chassis_link">
   <inertial>
     <origin rpy="0 0 0" xyz="1.04282e-06 0.07307 0.1816"/>
@@ -15,5 +21,5 @@
     <origin rpy="0 0 0" xyz="0 0 0"/>
     <geometry>
-      <mesh filename="package://ngeeann_av_description/meshes/base_link.stl" scale="0.001 0.001 0.001"/>
+      <mesh filename="package://ngeeann_av_description/meshes/chassis_link.stl" scale="0.001 0.001 0.001"/>
     </geometry>
     <material name="silver"/>
@@ -22,5 +28,5 @@
     <origin rpy="0 0 0" xyz="0 0 0"/>
     <geometry>
-      <mesh filename="package://ngeeann_av_description/meshes/base_link.stl" scale="0.001 0.001 0.001"/>
+      <mesh filename="package://ngeeann_av_description/meshes/chassis_link.stl" scale="0.001 0.001 0.001"/>
     </geometry>
   </collision>
@@ -122,5 +128,5 @@
 <joint name="br_axle" type="continuous">
   <origin rpy="0 0 0" xyz="0.8750 -1.013637 -0.144363"/>
-  <parent link="base_link"/>
+  <parent link="chassis_link"/>
   <child link="br_1"/>
   <axis xyz="-1.0 0.0 0.0"/>
@@ -128,5 +134,5 @@
 <joint name="bl_axle" type="continuous">
   <origin rpy="0 0 0" xyz="-0.8750 -1.013637 -0.144363"/>
-  <parent link="base_link"/>
+  <parent link="chassis_link"/>
   <child link="bl_1"/>
   <axis xyz="-1.0 0.0 0.0"/>
@@ -146,5 +152,5 @@
 <joint name="r_steer" type="revolute">
   <origin rpy="0 0 0" xyz="0.8250 1.517363 -0.144363"/>
-  <parent link="base_link"/>
+  <parent link="chassis_link"/>
   <child link="r_steer_1"/>
   <axis xyz="0.0 0.0 1.0"/>
@@ -154,5 +160,5 @@
 <joint name="l_steer" type="revolute">
   <origin rpy="0 0 0" xyz="-0.8250 1.517363 -0.144363"/>
-  <parent link="base_link"/>
+  <parent link="chassis_link"/>
   <child link="l_steer_1"/>
   <axis xyz="0.0 0.0 1.0"/>

Commit message: My way

File: ngeeann_av_description/urdf/camera.xacro (robot description, xacro)
@@ -12,5 +12,5 @@
       <origin xyz="0 0 0" rpy="0 0 0"/>
       <geometry>
-				<box size="0.05 0.05 0.05"/>
+			<box size="0.05 0.05 0.05"/>
       </geometry>
     </collision>
@@ -18,8 +18,8 @@
       <origin xyz="0 0 0" rpy="0 0 0"/>
       <geometry>
-				<box size="0.05 0.05 0.05"/>
+			<box size="0.05 0.05 0.05"/>
       </geometry>
       <material name="red">
-				<color rgba="1 0 0 1"/>
+			<color rgba="1 0 0 1"/>
       </material>
     </visual>
