Commit message: Add files via upload

File: ngeeann_av_description/urdf/ngeeann_av.xacro (robot description, xacro)
@@ -24,12 +24,32 @@
   </collision>
 </link>
+<link name="bl_1">
+  <inertial>
+    <origin rpy="0 0 0" xyz="0.037736 1.59295e-07 -1.59295e-07"/>
+    <mass value="24.5"/>
+    <inertia ixx="1.845139" ixy="-0.0" ixz="0.0" iyy="1.049606" iyz="0.0" izz="1.049606"/>
+  </inertial>
+  <visual>
+    <origin rpy="0 0 0" xyz="0.874999 1.013637 0.144363"/>
+    <geometry>
+      <mesh filename="package://ngeeann_av_description/meshes/bl_1.stl" scale="0.001 0.001 0.001"/>
+    </geometry>
+    <material name="darkgrey"/>
+  </visual>
+  <collision>
+    <origin rpy="0 0 0" xyz="0.874999 1.013637 0.144363"/>
+    <geometry>
+      <mesh filename="package://ngeeann_av_description/meshes/bl_1.stl" scale="0.001 0.001 0.001"/>
+    </geometry>
+  </collision>
+</link>
 <link name="br_1">
   <inertial>
-    <origin rpy="0 0 0" xyz="-0.03773558708170954 1.5929496499644813e-07 -1.5929501642752975e-07"/>
-    <mass value="24.339605554758485"/>
-    <inertia ixx="1.845139" ixy="-0.0" ixz="-0.0" iyy="1.049606" iyz="0.0" izz="1.049606"/>
-  </inertial>
-  <visual>
-    <origin rpy="0 0 0" xyz="-0.875001 1.013637 0.144363"/>
+    <origin rpy="0 0 0" xyz="0.037736 1.59295e-07 -1.59295e-07"/>
+    <mass value="24.5"/>
+    <inertia ixx="1.845139" ixy="-0.0" ixz="0.0" iyy="1.049606" iyz="0.0" izz="1.049606"/>
+  </inertial>
+  <visual>
+    <origin rpy="0 0 0" xyz="-0.874999 1.013637 0.144363"/>
     <geometry>
       <mesh filename="package://ngeeann_av_description/meshes/br_1.stl" scale="0.001 0.001 0.001"/>
@@ -38,5 +58,5 @@
   </visual>
   <collision>
-    <origin rpy="0 0 0" xyz="-0.875001 1.013637 0.144363"/>
+    <origin rpy="0 0 0" xyz="-0.874999 1.013637 0.144363"/>
     <geometry>
       <mesh filename="package://ngeeann_av_description/meshes/br_1.stl" scale="0.001 0.001 0.001"/>
@@ -44,21 +64,21 @@
   </collision>
 </link>
-<link name="bl_1">
-  <inertial>
-    <origin rpy="0 0 0" xyz="0.03773572073363374 1.5929503027756198e-07 -1.5929501642752975e-07"/>
-    <mass value="24.339605554758485"/>
-    <inertia ixx="1.845139" ixy="-0.0" ixz="0.0" iyy="1.049606" iyz="0.0" izz="1.049606"/>
-  </inertial>
-  <visual>
-    <origin rpy="0 0 0" xyz="0.874999 1.013637 0.144363"/>
-    <geometry>
-      <mesh filename="package://ngeeann_av_description/meshes/bl_1.stl" scale="0.001 0.001 0.001"/>
-    </geometry>
-    <material name="darkgrey"/>
-  </visual>
-  <collision>
-    <origin rpy="0 0 0" xyz="0.874999 1.013637 0.144363"/>
-    <geometry>
-      <mesh filename="package://ngeeann_av_description/meshes/bl_1.stl" scale="0.001 0.001 0.001"/>
+<link name="fl_1">
+  <inertial>
+    <origin rpy="0 0 0" xyz="0.037736 1.59295e-07 -1.59295e-07"/>
+    <mass value="24.5"/>
+    <inertia ixx="1.845139" ixy="-0.0" ixz="0.0" iyy="1.049606" iyz="0.0" izz="1.049606"/>
+  </inertial>
+  <visual>
+    <origin rpy="0 0 0" xyz="0.874999 -1.517363 0.144363"/>
+    <geometry>
+      <mesh filename="package://ngeeann_av_description/meshes/fl_1.stl" scale="0.001 0.001 0.001"/>
+    </geometry>
+    <material name="darkgrey"/>
+  </visual>
+  <collision>
+    <origin rpy="0 0 0" xyz="0.874999 -1.517363 0.144363"/>
+    <geometry>
+      <mesh filename="package://ngeeann_av_description/meshes/fl_1.stl" scale="0.001 0.001 0.001"/>
     </geometry>
   </collision>
@@ -66,10 +86,10 @@
 <link name="fr_1">
   <inertial>
-    <origin rpy="0 0 0" xyz="-0.03773558708161029 1.5929496499644813e-07 -1.5929500610245562e-07"/>
-    <mass value="24.339605554758485"/>
-    <inertia ixx="1.845139" ixy="-0.0" ixz="-0.0" iyy="1.049606" iyz="0.0" izz="1.049606"/>
-  </inertial>
-  <visual>
-    <origin rpy="0 0 0" xyz="-0.875001 -1.517363 0.144363"/>
+    <origin rpy="0 0 0" xyz="0.037736 1.59295e-07 -1.59295e-07"/>
+    <mass value="24.5"/>
+    <inertia ixx="1.845139" ixy="-0.0" ixz="0.0" iyy="1.049606" iyz="0.0" izz="1.049606"/>
+  </inertial>
+  <visual>
+    <origin rpy="0 0 0" xyz="-0.874999 -1.517363 0.144363"/>
     <geometry>
       <mesh filename="package://ngeeann_av_description/meshes/fr_1.stl" scale="0.001 0.001 0.001"/>
@@ -78,27 +98,7 @@
   </visual>
   <collision>
-    <origin rpy="0 0 0" xyz="-0.875001 -1.517363 0.144363"/>
+    <origin rpy="0 0 0" xyz="-0.874999 -1.517363 0.144363"/>
     <geometry>
       <mesh filename="package://ngeeann_av_description/meshes/fr_1.stl" scale="0.001 0.001 0.001"/>
-    </geometry>
-  </collision>
-</link>
-<link name="fl_1">
-  <inertial>
-    <origin rpy="0 0 0" xyz="0.037735720733733547 1.5929503005551737e-07 -1.5929500610245562e-07"/>
-    <mass value="24.339605554758485"/>
-    <inertia ixx="1.845139" ixy="-0.0" ixz="0.0" iyy="1.049606" iyz="0.0" izz="1.049606"/>
-  </inertial>
-  <visual>
-    <origin rpy="0 0 0" xyz="0.874999 -1.517363 0.144363"/>
-    <geometry>
-      <mesh filename="package://ngeeann_av_description/meshes/fl_1.stl" scale="0.001 0.001 0.001"/>
-    </geometry>
-    <material name="darkgrey"/>
-  </visual>
-  <collision>
-    <origin rpy="0 0 0" xyz="0.874999 -1.517363 0.144363"/>
-    <geometry>
-      <mesh filename="package://ngeeann_av_description/meshes/fl_1.stl" scale="0.001 0.001 0.001"/>
     </geometry>
   </collision>
@@ -131,5 +131,5 @@
   </inertial>
   <visual>
-    <origin rpy="0 0 0" xyz="0.824999 -1.517363 0.144363"/>
+    <origin rpy="0 0 0" xyz="0.825001 -1.517363 0.144363"/>
     <geometry>
       <mesh filename="package://ngeeann_av_description/meshes/l_steer_1.stl" scale="0.001 0.001 0.001"/>
@@ -138,5 +138,5 @@
   </visual>
   <collision>
-    <origin rpy="0 0 0" xyz="0.824999 -1.517363 0.144363"/>
+    <origin rpy="0 0 0" xyz="0.825001 -1.517363 0.144363"/>
     <geometry>
       <mesh filename="package://ngeeann_av_description/meshes/l_steer_1.stl" scale="0.001 0.001 0.001"/>
@@ -148,5 +148,5 @@
   <parent link="base_link"/>
   <child link="br_1"/>
-  <axis xyz="1.0 -0.0 -0.0"/>
+  <axis xyz="-1.0 0.0 0.0"/>
 </joint>
 <joint name="bl_axle" type="continuous">
@@ -160,5 +160,5 @@
   <parent link="r_steer_1"/>
   <child link="fr_1"/>
-  <axis xyz="1.0 -0.0 -0.0"/>
+  <axis xyz="-1.0 -0.0 -0.0"/>
 </joint>
 <joint name="fl_axle" type="continuous">

Commit message: Added camera sensor w/ some clean up

File: ngeeann_av_description/urdf/ngeeann_av.xacro (robot description, xacro)
@@ -4,4 +4,7 @@
 <xacro:include filename="$(find ngeeann_av_description)/urdf/ngeeann_av.trans" />
 <xacro:include filename="$(find ngeeann_av_description)/urdf/ngeeann_av.gazebo" />
+<xacro:include filename="$(find ngeeann_av_description)/urdf/hokuyo.xacro" />
+<xacro:include filename="$(find ngeeann_av_description)/urdf/camera.xacro" />
+<xacro:property name="camera_link" value="0.05" />
 <link name="base_link">
   <inertial>
@@ -24,8 +27,28 @@
   </collision>
 </link>
+<link name="br_1">
+  <inertial>
+    <origin rpy="0 0 0" xyz="-0.03773558708170954 1.5929496499644813e-07 -1.5929501642752975e-07"/>
+    <mass value="24.339605554758485"/>
+    <inertia ixx="1.845139" ixy="-0.0" ixz="-0.0" iyy="1.049606" iyz="0.0" izz="1.049606"/>
+  </inertial>
+  <visual>
+    <origin rpy="0 0 0" xyz="-0.875001 1.013637 0.144363"/>
+    <geometry>
+      <mesh filename="package://ngeeann_av_description/meshes/br_1.stl" scale="0.001 0.001 0.001"/>
+    </geometry>
+    <material name="darkgrey"/>
+  </visual>
+  <collision>
+    <origin rpy="0 0 0" xyz="-0.875001 1.013637 0.144363"/>
+    <geometry>
+      <mesh filename="package://ngeeann_av_description/meshes/br_1.stl" scale="0.001 0.001 0.001"/>
+    </geometry>
+  </collision>
+</link>
 <link name="bl_1">
   <inertial>
-    <origin rpy="0 0 0" xyz="0.037736 1.59295e-07 -1.59295e-07"/>
-    <mass value="24.5"/>
+    <origin rpy="0 0 0" xyz="0.03773572073363374 1.5929503027756198e-07 -1.5929501642752975e-07"/>
+    <mass value="24.339605554758485"/>
     <inertia ixx="1.845139" ixy="-0.0" ixz="0.0" iyy="1.049606" iyz="0.0" izz="1.049606"/>
   </inertial>
@@ -44,21 +67,21 @@
   </collision>
 </link>
-<link name="br_1">
+<link name="fr_1">
   <inertial>
-    <origin rpy="0 0 0" xyz="0.037736 1.59295e-07 -1.59295e-07"/>
-    <mass value="24.5"/>
-    <inertia ixx="1.845139" ixy="-0.0" ixz="0.0" iyy="1.049606" iyz="0.0" izz="1.049606"/>
+    <origin rpy="0 0 0" xyz="-0.03773558708161029 1.5929496499644813e-07 -1.5929500610245562e-07"/>
+    <mass value="24.339605554758485"/>
+    <inertia ixx="1.845139" ixy="-0.0" ixz="-0.0" iyy="1.049606" iyz="0.0" izz="1.049606"/>
   </inertial>
   <visual>
-    <origin rpy="0 0 0" xyz="-0.874999 1.013637 0.144363"/>
+    <origin rpy="0 0 0" xyz="-0.875001 -1.517363 0.144363"/>
     <geometry>
-      <mesh filename="package://ngeeann_av_description/meshes/br_1.stl" scale="0.001 0.001 0.001"/>
+      <mesh filename="package://ngeeann_av_description/meshes/fr_1.stl" scale="0.001 0.001 0.001"/>
     </geometry>
     <material name="darkgrey"/>
   </visual>
   <collision>
-    <origin rpy="0 0 0" xyz="-0.874999 1.013637 0.144363"/>
+    <origin rpy="0 0 0" xyz="-0.875001 -1.517363 0.144363"/>
     <geometry>
-      <mesh filename="package://ngeeann_av_description/meshes/br_1.stl" scale="0.001 0.001 0.001"/>
+      <mesh filename="package://ngeeann_av_description/meshes/fr_1.stl" scale="0.001 0.001 0.001"/>
     </geometry>
   </collision>
@@ -66,6 +89,6 @@
 <link name="fl_1">
   <inertial>
-    <origin rpy="0 0 0" xyz="0.037736 1.59295e-07 -1.59295e-07"/>
-    <mass value="24.5"/>
+    <origin rpy="0 0 0" xyz="0.037735720733733547 1.5929503005551737e-07 -1.5929500610245562e-07"/>
+    <mass value="24.339605554758485"/>
     <inertia ixx="1.845139" ixy="-0.0" ixz="0.0" iyy="1.049606" iyz="0.0" izz="1.049606"/>
   </inertial>
@@ -81,24 +104,4 @@
     <geometry>
       <mesh filename="package://ngeeann_av_description/meshes/fl_1.stl" scale="0.001 0.001 0.001"/>
-    </geometry>
-  </collision>
-</link>
-<link name="fr_1">
-  <inertial>
-    <origin rpy="0 0 0" xyz="0.037736 1.59295e-07 -1.59295e-07"/>
-    <mass value="24.5"/>
-    <inertia ixx="1.845139" ixy="-0.0" ixz="0.0" iyy="1.049606" iyz="0.0" izz="1.049606"/>
-  </inertial>
-  <visual>
-    <origin rpy="0 0 0" xyz="-0.874999 -1.517363 0.144363"/>
-    <geometry>
-      <mesh filename="package://ngeeann_av_description/meshes/fr_1.stl" scale="0.001 0.001 0.001"/>
-    </geometry>
-    <material name="darkgrey"/>
-  </visual>
-  <collision>
-    <origin rpy="0 0 0" xyz="-0.874999 -1.517363 0.144363"/>
-    <geometry>
-      <mesh filename="package://ngeeann_av_description/meshes/fr_1.stl" scale="0.001 0.001 0.001"/>
     </geometry>
   </collision>
@@ -131,5 +134,5 @@
   </inertial>
   <visual>
-    <origin rpy="0 0 0" xyz="0.825001 -1.517363 0.144363"/>
+    <origin rpy="0 0 0" xyz="0.824999 -1.517363 0.144363"/>
     <geometry>
       <mesh filename="package://ngeeann_av_description/meshes/l_steer_1.stl" scale="0.001 0.001 0.001"/>
@@ -138,5 +141,5 @@
   </visual>
   <collision>
-    <origin rpy="0 0 0" xyz="0.825001 -1.517363 0.144363"/>
+    <origin rpy="0 0 0" xyz="0.824999 -1.517363 0.144363"/>
     <geometry>
       <mesh filename="package://ngeeann_av_description/meshes/l_steer_1.stl" scale="0.001 0.001 0.001"/>
@@ -148,5 +151,5 @@
   <parent link="base_link"/>
   <child link="br_1"/>
-  <axis xyz="-1.0 0.0 0.0"/>
+  <axis xyz="1.0 -0.0 -0.0"/>
 </joint>
 <joint name="bl_axle" type="continuous">
@@ -160,5 +163,5 @@
   <parent link="r_steer_1"/>
   <child link="fr_1"/>
-  <axis xyz="-1.0 -0.0 -0.0"/>
+  <axis xyz="1.0 -0.0 -0.0"/>
 </joint>
 <joint name="fl_axle" type="continuous">
@@ -182,29 +185,3 @@
   <limit effort="1000.0" lower="-0.95" upper="0.95" velocity="5"/>
 </joint>
-<!-- Hokuyo Laser -->
-<joint name="hokuyo_joint" type="fixed">
-  <axis xyz="0 1 0" />
-  <origin xyz="0 2.34 0.24" rpy="0 0 1.5708"/>
-  <parent link="base_link"/>
-  <child link="hokuyo_link"/>
-</joint>
-<link name="hokuyo_link">
-  <collision>
-    <origin xyz="0 0 0" rpy="0 0 0"/>
-    <geometry>
-      <box size="0.05 0.05 0.05"/>
-    </geometry>
-  </collision>
-  <visual>
-    <origin xyz="0 0 0" rpy="0 0 0"/>
-    <geometry>
-      <mesh filename="package://ngeeann_av_description/meshes/hokuyo.dae"/>
-    </geometry>
-  </visual>
-  <inertial>
-    <mass value="1e-5" />
-    <origin xyz="0 0 0" rpy="0 0 0"/>
-    <inertia ixx="1e-6" ixy="0" ixz="0" iyy="1e-6" iyz="0" izz="1e-6" />
-  </inertial>
-</link>
 </robot>

Commit message: Update ngeeann_av.xacro

File: ngeeann_av_description/urdf/ngeeann_av.xacro (robot description, xacro)
@@ -6,9 +6,10 @@
 <xacro:include filename="$(find ngeeann_av_description)/urdf/hokuyo.xacro" />
 <xacro:include filename="$(find ngeeann_av_description)/urdf/camera.xacro" />
+<xacro:property name="camera_link" value="0.05" />
 <link name="base_link">
   <inertial>
-    <origin rpy="0 0 0" xyz="1.0428176421109296e-06 0.07306931261625653 0.18163727113784936"/>
-    <mass value="1577.05203547754"/>
-    <inertia ixx="1997.85793" ixy="-3e-05" ixz="-1e-06" iyy="442.769208" iyz="62.520613" izz="2238.052394"/>
+    <origin rpy="0 0 0" xyz="1.04282e-06 0.07307 0.1816"/>
+    <mass value="1580"/>
+    <inertia ixx="1997.8579" ixy="-3e-05" ixz="-1e-06" iyy="442.7692" iyz="62.5206" izz="2238.0524"/>
   </inertial>
   <visual>
@@ -28,10 +29,10 @@
 <link name="br_1">
   <inertial>
-    <origin rpy="0 0 0" xyz="-0.03773558708170954 1.5929496499644813e-07 -1.5929501642752975e-07"/>
-    <mass value="24.339605554758485"/>
+    <origin rpy="0 0 0" xyz="-0.0377 1.5929e-07 -1.5929e-07"/>
+    <mass value="24.5"/>
     <inertia ixx="1.845139" ixy="-0.0" ixz="-0.0" iyy="1.049606" iyz="0.0" izz="1.049606"/>
   </inertial>
   <visual>
-    <origin rpy="0 0 0" xyz="-0.875001 1.013637 0.144363"/>
+    <origin rpy="0 0 0" xyz="-0.8750 1.0136 0.1444"/>
     <geometry>
       <mesh filename="package://ngeeann_av_description/meshes/br_1.stl" scale="0.001 0.001 0.001"/>
@@ -40,5 +41,5 @@
   </visual>
   <collision>
-    <origin rpy="0 0 0" xyz="-0.875001 1.013637 0.144363"/>
+    <origin rpy="0 0 0" xyz="-0.8750 1.0136 0.1444"/>
     <geometry>
       <mesh filename="package://ngeeann_av_description/meshes/br_1.stl" scale="0.001 0.001 0.001"/>
@@ -48,10 +49,10 @@
 <link name="bl_1">
   <inertial>
-    <origin rpy="0 0 0" xyz="0.03773572073363374 1.5929503027756198e-07 -1.5929501642752975e-07"/>
-    <mass value="24.339605554758485"/>
-    <inertia ixx="1.845139" ixy="-0.0" ixz="0.0" iyy="1.049606" iyz="0.0" izz="1.049606"/>
+    <origin rpy="0 0 0" xyz="-0.0377 1.5929e-07 -1.5929e-07"/>
+    <mass value="24.5"/>
+    <inertia ixx="1.845139" ixy="-0.0" ixz="-0.0" iyy="1.049606" iyz="0.0" izz="1.049606"/>
   </inertial>
   <visual>
-    <origin rpy="0 0 0" xyz="0.874999 1.013637 0.144363"/>
+    <origin rpy="0 0 0" xyz="0.8750 1.0136 0.1444"/>
     <geometry>
       <mesh filename="package://ngeeann_av_description/meshes/bl_1.stl" scale="0.001 0.001 0.001"/>
@@ -60,5 +61,5 @@
   </visual>
   <collision>
-    <origin rpy="0 0 0" xyz="0.874999 1.013637 0.144363"/>
+    <origin rpy="0 0 0" xyz="0.8750 1.0136 0.1444"/>
     <geometry>
       <mesh filename="package://ngeeann_av_description/meshes/bl_1.stl" scale="0.001 0.001 0.001"/>
@@ -68,10 +69,10 @@
 <link name="fr_1">
   <inertial>
-    <origin rpy="0 0 0" xyz="-0.03773558708161029 1.5929496499644813e-07 -1.5929500610245562e-07"/>
-    <mass value="24.339605554758485"/>
+    <origin rpy="0 0 0" xyz="-0.0377 1.5929e-07 -1.5929e-07"/>
+    <mass value="24.5"/>
     <inertia ixx="1.845139" ixy="-0.0" ixz="-0.0" iyy="1.049606" iyz="0.0" izz="1.049606"/>
   </inertial>
   <visual>
-    <origin rpy="0 0 0" xyz="-0.875001 -1.517363 0.144363"/>
+    <origin rpy="0 0 0" xyz="-0.8750 -1.5174 0.1444"/>
     <geometry>
       <mesh filename="package://ngeeann_av_description/meshes/fr_1.stl" scale="0.001 0.001 0.001"/>
@@ -80,5 +81,5 @@
   </visual>
   <collision>
-    <origin rpy="0 0 0" xyz="-0.875001 -1.517363 0.144363"/>
+    <origin rpy="0 0 0" xyz="-0.8750 -1.5174 0.1444"/>
     <geometry>
       <mesh filename="package://ngeeann_av_description/meshes/fr_1.stl" scale="0.001 0.001 0.001"/>
@@ -88,10 +89,10 @@
 <link name="fl_1">
   <inertial>
-    <origin rpy="0 0 0" xyz="0.037735720733733547 1.5929503005551737e-07 -1.5929500610245562e-07"/>
-    <mass value="24.339605554758485"/>
-    <inertia ixx="1.845139" ixy="-0.0" ixz="0.0" iyy="1.049606" iyz="0.0" izz="1.049606"/>
+    <origin rpy="0 0 0" xyz="-0.0377 1.5929e-07 -1.5929e-07"/>
+    <mass value="24.5"/>
+    <inertia ixx="1.845139" ixy="-0.0" ixz="-0.0" iyy="1.049606" iyz="0.0" izz="1.049606"/>
   </inertial>
   <visual>
-    <origin rpy="0 0 0" xyz="0.874999 -1.517363 0.144363"/>
+    <origin rpy="0 0 0" xyz="0.8750 -1.5174 0.1444"/>
     <geometry>
       <mesh filename="package://ngeeann_av_description/meshes/fl_1.stl" scale="0.001 0.001 0.001"/>
@@ -100,5 +101,5 @@
   </visual>
   <collision>
-    <origin rpy="0 0 0" xyz="0.874999 -1.517363 0.144363"/>
+    <origin rpy="0 0 0" xyz="0.8750 -1.5174 0.1444"/>
     <geometry>
       <mesh filename="package://ngeeann_av_description/meshes/fl_1.stl" scale="0.001 0.001 0.001"/>
@@ -108,50 +109,24 @@
 <link name="r_steer_1">
   <inertial>
-    <origin rpy="0 0 0" xyz="0.0033805898024475978 1.5929497432232154e-07 0.021619317728612572"/>
-    <mass value="0.2193706942019361"/>
-    <inertia ixx="0.000163" ixy="-0.0" ixz="3e-06" iyy="0.000202" iyz="0.0" izz="0.000288"/>
+    <origin rpy="0 0 0" xyz="0.003381 1.5929e-07 0.02162"/>
+    <mass value="1"/>
+    <inertia ixx="1.0" ixy="0.0" ixz="0.0" iyy="1.0" iyz="0.0" izz="1.0"/>
   </inertial>
-  <visual>
-    <origin rpy="0 0 0" xyz="-0.825001 -1.517363 0.144363"/>
-    <geometry>
-      <mesh filename="package://ngeeann_av_description/meshes/r_steer_1.stl" scale="0.001 0.001 0.001"/>
-    </geometry>
-    <material name="darkgrey"/>
-  </visual>
-  <collision>
-    <origin rpy="0 0 0" xyz="-0.825001 -1.517363 0.144363"/>
-    <geometry>
-      <mesh filename="package://ngeeann_av_description/meshes/r_steer_1.stl" scale="0.001 0.001 0.001"/>
-    </geometry>
-  </collision>
 </link>
 <link name="l_steer_1">
   <inertial>
-    <origin rpy="0 0 0" xyz="-0.0033804561503246733 1.5929503982548e-07 0.021619317728612572"/>
-    <mass value="0.2193706942019361"/>
-    <inertia ixx="0.000163" ixy="-0.0" ixz="-3e-06" iyy="0.000202" iyz="0.0" izz="0.000288"/>
+    <origin rpy="0 0 0" xyz="0.003381 1.5929e-07 0.02162"/>
+    <mass value="1"/>
+    <inertia ixx="1.0" ixy="0.0" ixz="0.0" iyy="1.0" iyz="0.0" izz="1.0"/>
   </inertial>
-  <visual>
-    <origin rpy="0 0 0" xyz="0.824999 -1.517363 0.144363"/>
-    <geometry>
-      <mesh filename="package://ngeeann_av_description/meshes/l_steer_1.stl" scale="0.001 0.001 0.001"/>
-    </geometry>
-    <material name="darkgrey"/>
-  </visual>
-  <collision>
-    <origin rpy="0 0 0" xyz="0.824999 -1.517363 0.144363"/>
-    <geometry>
-      <mesh filename="package://ngeeann_av_description/meshes/l_steer_1.stl" scale="0.001 0.001 0.001"/>
-    </geometry>
-  </collision>
 </link>
 <joint name="br_axle" type="continuous">
-  <origin rpy="0 0 0" xyz="0.875001 -1.013637 -0.144363"/>
+  <origin rpy="0 0 0" xyz="0.8750 -1.013637 -0.144363"/>
   <parent link="base_link"/>
   <child link="br_1"/>
-  <axis xyz="1.0 -0.0 -0.0"/>
+  <axis xyz="-1.0 0.0 0.0"/>
 </joint>
 <joint name="bl_axle" type="continuous">
-  <origin rpy="0 0 0" xyz="-0.874999 -1.013637 -0.144363"/>
+  <origin rpy="0 0 0" xyz="-0.8750 -1.013637 -0.144363"/>
   <parent link="base_link"/>
   <child link="bl_1"/>
@@ -162,5 +137,5 @@
   <parent link="r_steer_1"/>
   <child link="fr_1"/>
-  <axis xyz="1.0 -0.0 -0.0"/>
+  <axis xyz="-1.0 0.0 0.0"/>
 </joint>
 <joint name="fl_axle" type="continuous">
@@ -170,30 +145,18 @@
   <axis xyz="-1.0 0.0 0.0"/>
 </joint>
-<joint name="fr_steer" type="revolute">
-  <origin rpy="0 0 0" xyz="0.825001 1.517363 -0.144363"/>
+<joint name="r_steer" type="revolute">
+  <origin rpy="0 0 0" xyz="0.8250 1.517363 -0.144363"/>
   <parent link="base_link"/>
   <child link="r_steer_1"/>
-  <axis xyz="-0.0 -0.0 1.0"/>
+  <axis xyz="0.0 0.0 1.0"/>
+  <dynamics damping="0.7" friction="0.7"/>
   <limit effort="1000.0" lower="-0.95" upper="0.95" velocity="5"/>
 </joint>
-<joint name="fl_steer" type="revolute">
-  <origin rpy="0 0 0" xyz="-0.824999 1.517363 -0.144363"/>
+<joint name="l_steer" type="revolute">
+  <origin rpy="0 0 0" xyz="-0.8250 1.517363 -0.144363"/>
   <parent link="base_link"/>
   <child link="l_steer_1"/>
-  <axis xyz="-0.0 -0.0 1.0"/>
-  <limit effort="1000.0" lower="-0.95" upper="0.95" velocity="5"/>
-</joint>
-<joint name="fr_steer" type="revolute">
-  <origin rpy="0 0 0" xyz="0.825001 1.517363 -0.144363"/>
-  <parent link="base_link"/>
-  <child link="r_steer_1"/>
-  <axis xyz="-0.0 -0.0 1.0"/>
-  <limit effort="1000.0" lower="-0.95" upper="0.95" velocity="5"/>
-</joint>
-<joint name="fl_steer" type="revolute">
-  <origin rpy="0 0 0" xyz="-0.824999 1.517363 -0.144363"/>
-  <parent link="base_link"/>
-  <child link="l_steer_1"/>
-  <axis xyz="-0.0 -0.0 1.0"/>
+  <axis xyz="0.0 0.0 1.0"/>
+  <dynamics damping="0.7" friction="0.7"/>
   <limit effort="1000.0" lower="-0.95" upper="0.95" velocity="5"/>
 </joint>

Commit message: Update ngeeann_av.xacro

File: ngeeann_av_description/urdf/ngeeann_av.xacro (robot description, xacro)
@@ -6,5 +6,4 @@
 <xacro:include filename="$(find ngeeann_av_description)/urdf/hokuyo.xacro" />
 <xacro:include filename="$(find ngeeann_av_description)/urdf/camera.xacro" />
-<xacro:property name="camera_link" value="0.05" />
 <link name="base_link">
   <inertial>

Commit message: ackerman_params.yaml added

File: ngeeann_av_description/urdf/ngeeann_av.xacro (robot description, xacro)
@@ -149,6 +149,6 @@
   <child link="r_steer_1"/>
   <axis xyz="0.0 0.0 1.0"/>
-  <dynamics damping="0.7" friction="0.7"/>
-  <limit effort="1000.0" lower="-0.95" upper="0.95" velocity="5"/>
+  <dynamics damping="0.01" friction="0.01"/>
+  <limit effort="1000.0" lower="-0.95" upper="0.95" velocity="100"/>
 </joint>
 <joint name="l_steer" type="revolute">
@@ -157,6 +157,6 @@
   <child link="l_steer_1"/>
   <axis xyz="0.0 0.0 1.0"/>
-  <dynamics damping="0.7" friction="0.7"/>
-  <limit effort="1000.0" lower="-0.95" upper="0.95" velocity="5"/>
+  <dynamics damping="0.01" friction="0.01"/>
+  <limit effort="1000.0" lower="-0.95" upper="0.95" velocity="100"/>
 </joint>
 </robot>
