Commit message: most useless update, added spoiler

File: ngeeann_av_description/urdf/ngeeann_av.xacro (robot description, xacro)
@@ -29,4 +29,24 @@
     <geometry>
       <mesh filename="package://ngeeann_av_description/meshes/chassis_link.stl" scale="0.001 0.001 0.001"/>
+    </geometry>
+  </collision>
+</link>
+<joint name="spoiler_joint" type="fixed">
+  <origin xyz="0 0.05 -0.05" rpy="1.5708 0 3.14159" />
+  <parent link="chassis_link"/>
+  <child link="spoiler_link"/>
+</joint>
+<link name="spoiler_link">
+  <visual>
+    <origin rpy="0 0 0" xyz="0 0 0"/>
+    <geometry>
+      <mesh filename="package://ngeeann_av_description/meshes/spoiler.stl" scale="0.001 0.001 0.001"/>
+    </geometry>
+    <material name="silver"/>
+  </visual>
+  <collision>
+    <origin rpy="0 0 0" xyz="0 0 0"/>
+    <geometry>
+      <mesh filename="package://ngeeann_av_description/meshes/spoiler.stl" scale="0.001 0.001 0.001"/>
     </geometry>
   </collision>

Commit message: useless mods #2: the car is more aero now

File: ngeeann_av_description/urdf/ngeeann_av.xacro (robot description, xacro)
@@ -19,5 +19,5 @@
   </inertial>
   <visual>
-    <origin rpy="0 0 0" xyz="0 0 0"/>
+    <origin rpy="1.5708 0 3.14159" xyz="0 0.04 -0.05"/>
     <geometry>
       <mesh filename="package://ngeeann_av_description/meshes/chassis_link.stl" scale="0.001 0.001 0.001"/>

Commit message: nvm the car exploded when i drive so aero for another day

File: ngeeann_av_description/urdf/ngeeann_av.xacro (robot description, xacro)
@@ -19,5 +19,5 @@
   </inertial>
   <visual>
-    <origin rpy="1.5708 0 3.14159" xyz="0 0.04 -0.05"/>
+    <origin rpy="0 0 0" xyz="0 0 0"/>
     <geometry>
       <mesh filename="package://ngeeann_av_description/meshes/chassis_link.stl" scale="0.001 0.001 0.001"/>
